Commit message: Updates for simulations autorun

File: urdf/projectile.urdf (robot description, URDF)
Before this commit: robot projectile, 1 links, 0 joints
Links:
- link projectile_link: geometry collision sphere radius=0.01; visual sphere radius=0.1

File: worlds/goals.sdf.xacro (robot description, xacro)
@@ -20,5 +20,5 @@
         </visual>
         <collision name='collision'>
-          <pose>0 0 ${sz*cz}</pose>
+          <pose>0 0 ${sz*cz/2}</pose>
           <geometry>
             <box>

File: worlds/obstacles.sdf.xacro (robot description, xacro)
@@ -342,5 +342,5 @@
         </visual>
         <collision name='collision'>
-          <pose>0 0 ${sz*cz}</pose>
+          <pose>0 0 ${sz*cz/2} 0 0 0</pose>
           <geometry>
             <!-- <mesh>
